File: ICM-42688-P/SV4_ICM.kicad_pcb (KiCad board)
At the start: 2 copper layers, 17.8 x 26.4 mm, 17 parts, among them U1 SuperMini nRF52840, U2 ICM-42688-P, U3 MMC5983MA

Commit message: - Added PCB push hole for easier disassembly - Increased pin push hole for SIM tools - Added disassembly slide to release battery tray - Added i2c pullups... I can't believe I forgot those. I already ordered the boards, too. Am I stupid??? - Increased height of button deflector to direct forces more inward - Added "mirror" on PCB for better light - Added photos of tracker
Parts:
- added R1: 10k, Resistor_SMD:R_0402_1005Metric, F.Cu at (146.8, 77.5)
- added R2: 10k, Resistor_SMD:R_0402_1005Metric, F.Cu at (146.3, 88.9)
Routing:
- net GND: track 20.8 -> 23.0 mm
- net +3V3: track 50.6 -> 52.2 mm
